Commit message: change names

File: source/magiclab_rl_lab/magiclab_rl_lab/data/robots/magicbot-Z1/urdf/MagicBotZ1.urdf (robot description, URDF)
Before this commit: robot MagicBotZ1, 31 links, 30 joints
Links:
- removed link LINK_ANKLE_PITCH_L
- removed link LINK_ANKLE_PITCH_R
- removed link LINK_ANKLE_ROLL_L
- removed link LINK_ANKLE_ROLL_R
- removed link LINK_FOOT_L
- removed link LINK_FOOT_R
- removed link LINK_HAND_L
- removed link LINK_HAND_R
- removed link LINK_HIP_PITCH_L
- removed link LINK_HIP_PITCH_R
- removed link LINK_HIP_ROLL_L
- removed link LINK_HIP_ROLL_R
- removed link LINK_HIP_YAW_L
- removed link LINK_HIP_YAW_R
- removed link LINK_KNEE_PITCH_L
- removed link LINK_KNEE_PITCH_R
- removed link LINK_TOE_L
- removed link LINK_TOE_R
- removed link link_hy
- removed link link_la1
- removed link link_la2
- removed link link_la3
- removed link link_la4
- removed link link_la5
- removed link link_ra1
- removed link link_ra2
- removed link link_ra3
- removed link link_ra4
- removed link link_ra5
- removed link link_wy
- added link head_link, mass 0.7987; visual mesh filename=../meshes/head_link.STL
- added link left_ankle_pitch_link, mass 0.048544; visual mesh filename=../meshes/left_ankle_pitch_link.STL
- added link left_ankle_roll_link, mass 0.7019; collision box size=0.21622 0.050 0.02; visual mesh filename=../meshes/left_ankle_roll_link.STL
- added link left_elbow_link, mass 1.48; collision mesh filename=../meshes/left_elbow_link.STL; visual mesh filename=../meshes/left_elbow_link.STL
- added link left_foot_link, mass 1e-12
- added link left_hand_palm_link, mass 1e-12
- added link left_hip_pitch_link, mass 1.5089; visual mesh filename=../meshes/left_hip_pitch_link.STL
- added link left_hip_roll_link, mass 1.9215; visual mesh filename=../meshes/left_hip_roll_link.STL
- added link left_hip_yaw_link, mass 0.9002; visual mesh filename=../meshes/left_hip_yaw_link.STL
- added link left_knee_link, mass 3.7275; collision mesh filename=../meshes/left_knee_link.STL; visual mesh filename=../meshes/left_knee_link.STL
- added link left_shoulder_pitch_link, mass 0.8939; visual mesh filename=../meshes/left_shoulder_pitch_link.STL
- added link left_shoulder_roll_link, mass 0.7787; visual mesh filename=../meshes/left_shoulder_roll_link.STL
- added link left_shoulder_yaw_link, mass 0.35928; visual mesh filename=../meshes/left_shoulder_yaw_link.STL
- added link left_toe_link, mass 1e-12
- added link left_wrist_yaw_link, mass 0.2728; collision mesh filename=../meshes/left_wrist_yaw_link.STL; visual mesh filename=../meshes/left_wrist_yaw_link.STL
- added link right_ankle_pitch_link, mass 0.048544; visual mesh filename=../meshes/right_ankle_pitch_link.STL
- added link right_ankle_roll_link, mass 0.70183; collision box size=0.21622 0.050 0.02; visual mesh filename=../meshes/right_ankle_roll_link.STL
- added link right_elbow_link, mass 1.48; collision mesh filename=../meshes/right_elbow_link.STL; visual mesh filename=../meshes/right_elbow_link.STL
- added link right_foot_link, mass 1e-12
- added link right_hand_palm_link, mass 1e-12
- added link right_hip_pitch_link, mass 1.5089; visual mesh filename=../meshes/right_hip_pitch_link.STL
- added link right_hip_roll_link, mass 1.9215; visual mesh filename=../meshes/right_hip_roll_link.STL
- added link right_hip_yaw_link, mass 0.9002; visual mesh filename=../meshes/right_hip_yaw_link.STL
- added link right_knee_link, mass 3.7292; collision mesh filename=../meshes/right_knee_link.STL; visual mesh filename=../meshes/right_knee_link.STL
- added link right_shoulder_pitch_link, mass 0.8976; visual mesh filename=../meshes/right_shoulder_pitch_link.STL
- added link right_shoulder_roll_link, mass 0.7868; visual mesh filename=../meshes/right_shoulder_roll_link.STL
- added link right_shoulder_yaw_link, mass 0.3593; visual mesh filename=../meshes/right_shoulder_yaw_link.STL
- added link right_toe_link, mass 1e-12
- added link right_wrist_yaw_link, mass 0.27279; collision mesh filename=../meshes/right_wrist_yaw_link.STL; visual mesh filename=../meshes/right_wrist_yaw_link.STL
- added link torso_link, mass 9.8779; collision mesh filename=../meshes/torso_link.STL; visual mesh filename=../meshes/torso_link.STL
Joints:
- removed joint JOINT_ANKLE_PITCH_L
- removed joint JOINT_ANKLE_PITCH_R
- removed joint JOINT_ANKLE_ROLL_L
- removed joint JOINT_ANKLE_ROLL_R
- removed joint JOINT_HIP_PITCH_L
- removed joint JOINT_HIP_PITCH_R
- removed joint JOINT_HIP_ROLL_L
- removed joint JOINT_HIP_ROLL_R
- removed joint JOINT_HIP_YAW_L
- removed joint JOINT_HIP_YAW_R
- removed joint JOINT_KNEE_PITCH_L
- removed joint JOINT_KNEE_PITCH_R
- removed joint JOINT_TOE_L
- removed joint JOINT_TOE_R
- removed joint J_FOOT_L
- removed joint J_FOOT_R
- removed joint J_HAND_L
- removed joint J_HAND_R
- removed joint joint_hy
- removed joint joint_la1
- removed joint joint_la2
- removed joint joint_la3
- removed joint joint_la4
- removed joint joint_la5
- removed joint joint_ra1
- removed joint joint_ra2
- removed joint joint_ra3
- removed joint joint_ra4
- removed joint joint_ra5
- removed joint joint_wy
- added joint head_joint: type fixed, parent torso_link, child head_link, origin xyz=0 0 0.4889 rpy=0 0 0, axis 0 0 1, limit lower=-0.6981 upper=0.6981 effort=50 velocity=15
- added joint left_ankle_pitch_joint: type revolute, parent left_knee_link, child left_ankle_pitch_link, origin xyz=0 0 -0.34 rpy=0 0 0, axis 0 1 0, limit lower=-0.873 upper=0.524 effort=50 velocity=15
- added joint left_ankle_roll_joint: type revolute, parent left_ankle_pitch_link, child left_ankle_roll_link, origin xyz=0 0 -0.018 rpy=0 0 0, axis 1 0 0, limit lower=-0.262 upper=0.262 effort=50 velocity=15
- added joint left_elbow_joint: type fixed, parent left_shoulder_yaw_link, child left_elbow_link, origin xyz=0.01924 0 -0.0979 rpy=0 0 0, axis 0 1 0, limit lower=-0.96 upper=2.0944 effort=50 velocity=14
- added joint left_foot_joint: type fixed, parent left_ankle_roll_link, child left_foot_link, origin xyz=-0. 0.000000 -0.0447600 rpy=0 0 0, axis 0 0 1
- added joint left_hand_palm_joint: type fixed, parent left_wrist_yaw_link, child left_hand_palm_link, origin xyz=0.138 0.000000 -0. rpy=0 0 0, axis 0 0 1
- added joint left_hip_pitch_joint: type revolute, parent pelvis, child left_hip_pitch_link, origin xyz=0 0.06875 0 rpy=0 0 0, axis 0 1 0, limit lower=-2.7925 upper=2.7925 effort=120 velocity=20
- added joint left_hip_roll_joint: type revolute, parent left_hip_pitch_link, child left_hip_roll_link, origin xyz=0 0.053724 -0.045579 rpy=0 0 0, axis 1 0 0, limit lower=-0.524 upper=2.967 effort=120 velocity=20
- added joint left_hip_yaw_joint: type revolute, parent left_hip_roll_link, child left_hip_yaw_link, origin xyz=-0.00084052 0 -0.1255 rpy=0 0 0, axis 0 0 1, limit lower=-2.7925 upper=2.7925 effort=120 velocity=20
- added joint left_knee_joint: type revolute, parent left_hip_yaw_link, child left_knee_link, origin xyz=-0.052111 0 -0.13729 rpy=0 0 0, axis 0 1 0, limit lower=0 upper=2.653 effort=120 velocity=20
- added joint left_shoulder_pitch_joint: type fixed, parent torso_link, child left_shoulder_pitch_link, origin xyz=0 0.11963 0.3208 rpy=0 0 0, axis 0 0.99255 -0.12187, limit lower=-2.88 upper=2.88 effort=50 velocity=14
- added joint left_shoulder_roll_joint: type fixed, parent left_shoulder_pitch_link, child left_shoulder_roll_link, origin xyz=0 0.047187 -0.013786 rpy=0 0 0, axis 1 0 0, limit lower=-0.175 upper=2.2515 effort=50 velocity=14
- added joint left_shoulder_yaw_joint: type fixed, parent left_shoulder_roll_link, child left_shoulder_yaw_link, origin xyz=0 0 -0.1171 rpy=0 0 0, axis 0 0 1, limit lower=-2.618 upper=2.618 effort=50 velocity=14
- added joint left_toe_joint: type fixed, parent left_foot_link, child left_toe_link, origin xyz=0.152 0 0 rpy=0 0 0, axis 0 1 0
- added joint left_wrist_yaw_joint: type fixed, parent left_elbow_link, child left_wrist_yaw_link, origin xyz=0.138 0 -0.017415 rpy=0 0 0, axis 1 0 0, limit lower=-2.618 upper=2.618 effort=50 velocity=14
- added joint right_ankle_pitch_joint: type revolute, parent right_knee_link, child right_ankle_pitch_link, origin xyz=0 0 -0.34 rpy=0 0 0, axis 0 1 0, limit lower=-0.873 upper=0.524 effort=50 velocity=15
- added joint right_ankle_roll_joint: type revolute, parent right_ankle_pitch_link, child right_ankle_roll_link, origin xyz=0 0 -0.018 rpy=0 0 0, axis 1 0 0, limit lower=-0.262 upper=0.262 effort=50 velocity=15
- added joint right_elbow_joint: type fixed, parent right_shoulder_yaw_link, child right_elbow_link, origin xyz=0.01924 0 -0.0979 rpy=0 0 0, axis 0 1 0, limit lower=-0.96 upper=2.0944 effort=50 velocity=14
- added joint right_foot_joint: type fixed, parent right_ankle_roll_link, child right_foot_link, origin xyz=0.000000 0.000000 -0.044760000 rpy=0 0 0, axis 0 0 1
- added joint right_hand_palm_joint: type fixed, parent right_wrist_yaw_link, child right_hand_palm_link, origin xyz=0.138 0.000000 0.0 rpy=0 0 0, axis 0 0 1
- added joint right_hip_pitch_joint: type revolute, parent pelvis, child right_hip_pitch_link, origin xyz=0 -0.06875 0 rpy=0 0 0, axis 0 1 0, limit lower=-2.7925 upper=2.7925 effort=120 velocity=20
- added joint right_hip_roll_joint: type revolute, parent right_hip_pitch_link, child right_hip_roll_link, origin xyz=0 -0.053724 -0.045579 rpy=0 0 0, axis 1 0 0, limit lower=-2.967 upper=0.524 effort=120 velocity=20
- added joint right_hip_yaw_joint: type revolute, parent right_hip_roll_link, child right_hip_yaw_link, origin xyz=-0.00050599 0.0029213 -0.12555 rpy=0 0 0, axis 0 0 1, limit lower=-2.7925 upper=2.7925 effort=120 velocity=20
- added joint right_knee_joint: type revolute, parent right_hip_yaw_link, child right_knee_link, origin xyz=-0.052111 0 -0.13729 rpy=0 0 0, axis 0 1 0, limit lower=0 upper=2.653 effort=120 velocity=20
- added joint right_shoulder_pitch_joint: type fixed, parent torso_link, child right_shoulder_pitch_link, origin xyz=0 -0.11963 0.3208 rpy=0 0 0, axis 0 0.99255 -0.12187, limit lower=-2.88 upper=2.88 effort=50 velocity=14
- added joint right_shoulder_roll_joint: type fixed, parent right_shoulder_pitch_link, child right_shoulder_roll_link, origin xyz=0 -0.047187 -0.013786 rpy=0 0 0, axis 1 0 0, limit lower=-2.2515 upper=0.175 effort=50 velocity=14
- added joint right_shoulder_yaw_joint: type fixed, parent right_shoulder_roll_link, child right_shoulder_yaw_link, origin xyz=0 0 -0.1171 rpy=0 0 0, axis 0 0 1, limit lower=-2.618 upper=2.618 effort=50 velocity=14
- added joint right_toe_joint: type fixed, parent right_foot_link, child right_toe_link, origin xyz=0.152 0 0 rpy=0 0 0, axis 1 0 0
- added joint right_wrist_yaw_joint: type fixed, parent right_elbow_link, child right_wrist_yaw_link, origin xyz=0.138 0 -0.017415 rpy=0 0 0, axis 1 0 0, limit lower=-2.618 upper=2.618 effort=50 velocity=14
- added joint waist_yaw_joint: type fixed, parent pelvis, child torso_link, origin xyz=0 0 0.0619 rpy=0 0 0, axis 0 0 1, limit lower=-2.79 upper=2.79 effort=120 velocity=20

File: source/magiclab_rl_lab/magiclab_rl_lab/data/robots/magicbot-Z1/urdf/MagicBotZ1_arm_ready_pos.urdf (robot description, URDF)
Before this commit: robot MagicBotZ1, 31 links, 30 joints
Links:
- removed link LINK_ANKLE_PITCH_L
- removed link LINK_ANKLE_PITCH_R
- removed link LINK_ANKLE_ROLL_L
- removed link LINK_ANKLE_ROLL_R
- removed link LINK_FOOT_L
- removed link LINK_FOOT_R
- removed link LINK_HAND_L
- removed link LINK_HAND_R
- removed link LINK_HIP_PITCH_L
- removed link LINK_HIP_PITCH_R
- removed link LINK_HIP_ROLL_L
- removed link LINK_HIP_ROLL_R
- removed link LINK_HIP_YAW_L
- removed link LINK_HIP_YAW_R
- removed link LINK_KNEE_PITCH_L
- removed link LINK_KNEE_PITCH_R
- removed link LINK_TOE_L
- removed link LINK_TOE_R
- removed link link_hy
- removed link link_la1
- removed link link_la2
- removed link link_la3
- removed link link_la4
- removed link link_la5
- removed link link_ra1
- removed link link_ra2
- removed link link_ra3
- removed link link_ra4
- removed link link_ra5
- removed link link_wy
- added link head_link, mass 0.7987; visual mesh filename=../meshes/head_link.STL
- added link left_ankle_pitch_link, mass 0.048544; visual mesh filename=../meshes/left_ankle_pitch_link.STL
- added link left_ankle_roll_link, mass 0.7019; collision box size=0.21622 0.050 0.02; visual mesh filename=../meshes/left_ankle_roll_link.STL
- added link left_elbow_link, mass 1.48; collision mesh filename=../meshes/left_elbow_link.STL; visual mesh filename=../meshes/left_elbow_link.STL
- added link left_foot_link, mass 1e-12
- added link left_hand_palm_link, mass 1e-12
- added link left_hip_pitch_link, mass 1.5089; visual mesh filename=../meshes/left_hip_pitch_link.STL
- added link left_hip_roll_link, mass 1.9215; visual mesh filename=../meshes/left_hip_roll_link.STL
- added link left_hip_yaw_link, mass 0.9002; visual mesh filename=../meshes/left_hip_yaw_link.STL
- added link left_knee_link, mass 3.7275; collision mesh filename=../meshes/left_knee_link.STL; visual mesh filename=../meshes/left_knee_link.STL
- added link left_shoulder_pitch_link, mass 0.8939; visual mesh filename=../meshes/left_shoulder_pitch_link.STL
- added link left_shoulder_roll_link, mass 0.7787; visual mesh filename=../meshes/left_shoulder_roll_link.STL
- added link left_shoulder_yaw_link, mass 0.35928; visual mesh filename=../meshes/left_shoulder_yaw_link.STL
- added link left_toe_link, mass 1e-12
- added link left_wrist_yaw_link, mass 0.2728; collision mesh filename=../meshes/left_wrist_yaw_link.STL; visual mesh filename=../meshes/left_wrist_yaw_link.STL
- added link right_ankle_pitch_link, mass 0.048544; visual mesh filename=../meshes/right_ankle_pitch_link.STL
- added link right_ankle_roll_link, mass 0.70183; collision box size=0.21622 0.050 0.02; visual mesh filename=../meshes/right_ankle_roll_link.STL
- added link right_elbow_link, mass 1.48; collision mesh filename=../meshes/right_elbow_link.STL; visual mesh filename=../meshes/right_elbow_link.STL
- added link right_foot_link, mass 1e-12
- added link right_hand_palm_link, mass 1e-12
- added link right_hip_pitch_link, mass 1.5089; visual mesh filename=../meshes/right_hip_pitch_link.STL
- added link right_hip_roll_link, mass 1.9215; visual mesh filename=../meshes/right_hip_roll_link.STL
- added link right_hip_yaw_link, mass 0.9002; visual mesh filename=../meshes/right_hip_yaw_link.STL
- added link right_knee_link, mass 3.7292; collision mesh filename=../meshes/right_knee_link.STL; visual mesh filename=../meshes/right_knee_link.STL
- added link right_shoulder_pitch_link, mass 0.8976; visual mesh filename=../meshes/right_shoulder_pitch_link.STL
- added link right_shoulder_roll_link, mass 0.7868; visual mesh filename=../meshes/right_shoulder_roll_link.STL
- added link right_shoulder_yaw_link, mass 0.3593; visual mesh filename=../meshes/right_shoulder_yaw_link.STL
- added link right_toe_link, mass 1e-12
- added link right_wrist_yaw_link, mass 0.27279; collision mesh filename=../meshes/right_wrist_yaw_link.STL; visual mesh filename=../meshes/right_wrist_yaw_link.STL
- added link torso_link, mass 9.8779; collision mesh filename=../meshes/torso_link.STL; visual mesh filename=../meshes/torso_link.STL
Joints:
- removed joint JOINT_ANKLE_PITCH_L
- removed joint JOINT_ANKLE_PITCH_R
- removed joint JOINT_ANKLE_ROLL_L
- removed joint JOINT_ANKLE_ROLL_R
- removed joint JOINT_HIP_PITCH_L
- removed joint JOINT_HIP_PITCH_R
- removed joint JOINT_HIP_ROLL_L
- removed joint JOINT_HIP_ROLL_R
- removed joint JOINT_HIP_YAW_L
- removed joint JOINT_HIP_YAW_R
- removed joint JOINT_KNEE_PITCH_L
- removed joint JOINT_KNEE_PITCH_R
- removed joint JOINT_TOE_L
- removed joint JOINT_TOE_R
- removed joint J_FOOT_L
- removed joint J_FOOT_R
- removed joint J_HAND_L
- removed joint J_HAND_R
- removed joint joint_hy
- removed joint joint_la1
- removed joint joint_la2
- removed joint joint_la3
- removed joint joint_la4
- removed joint joint_la5
- removed joint joint_ra1
- removed joint joint_ra2
- removed joint joint_ra3
- removed joint joint_ra4
- removed joint joint_ra5
- removed joint joint_wy
- added joint head_joint: type fixed, parent torso_link, child head_link, origin xyz=0 0 0.4889 rpy=0 0 0, axis 0 0 1, limit lower=-0.6981 upper=0.6981 effort=50 velocity=15
- added joint left_ankle_pitch_joint: type revolute, parent left_knee_link, child left_ankle_pitch_link, origin xyz=0 0 -0.34 rpy=0 0 0, axis 0 1 0, limit lower=-0.873 upper=0.524 effort=50 velocity=15
- added joint left_ankle_roll_joint: type revolute, parent left_ankle_pitch_link, child left_ankle_roll_link, origin xyz=0 0 -0.018 rpy=0 0 0, axis 1 0 0, limit lower=-0.262 upper=0.262 effort=50 velocity=15
- added joint left_elbow_joint: type fixed, parent left_shoulder_yaw_link, child left_elbow_link, origin xyz=0.01924 0 -0.0979 rpy=0 1 0, axis 0 1 0, limit lower=-0.96 upper=2.0944 effort=50 velocity=14
- added joint left_foot_joint: type fixed, parent left_ankle_roll_link, child left_foot_link, origin xyz=-0. 0.000000 -0.0447600 rpy=0 0 0, axis 0 0 1
- added joint left_hand_palm_joint: type fixed, parent left_wrist_yaw_link, child left_hand_palm_link, origin xyz=0.138 0.000000 -0. rpy=0 0 0, axis 0 0 1
- added joint left_hip_pitch_joint: type revolute, parent pelvis, child left_hip_pitch_link, origin xyz=0 0.06875 0 rpy=0 0 0, axis 0 1 0, limit lower=-2.7925 upper=2.7925 effort=120 velocity=20
- added joint left_hip_roll_joint: type revolute, parent left_hip_pitch_link, child left_hip_roll_link, origin xyz=0 0.053724 -0.045579 rpy=0 0 0, axis 1 0 0, limit lower=-0.524 upper=2.967 effort=120 velocity=20
- added joint left_hip_yaw_joint: type revolute, parent left_hip_roll_link, child left_hip_yaw_link, origin xyz=-0.00084052 0 -0.1255 rpy=0 0 0, axis 0 0 1, limit lower=-2.7925 upper=2.7925 effort=120 velocity=20
- added joint left_knee_joint: type revolute, parent left_hip_yaw_link, child left_knee_link, origin xyz=-0.052111 0 -0.13729 rpy=0 0 0, axis 0 1 0, limit lower=0 upper=2.653 effort=120 velocity=20
- added joint left_shoulder_pitch_joint: type fixed, parent torso_link, child left_shoulder_pitch_link, origin xyz=0 0.11963 0.3208 rpy=0 0.2 0, axis 0 0.99255 -0.12187, limit lower=-2.88 upper=2.88 effort=50 velocity=14
- added joint left_shoulder_roll_joint: type fixed, parent left_shoulder_pitch_link, child left_shoulder_roll_link, origin xyz=0 0.047187 -0.013786 rpy=0.15 0 0, axis 1 0 0, limit lower=-0.175 upper=2.2515 effort=50 velocity=14
- added joint left_shoulder_yaw_joint: type fixed, parent left_shoulder_roll_link, child left_shoulder_yaw_link, origin xyz=0 0 -0.1171 rpy=0 0 0, axis 0 0 1, limit lower=-2.618 upper=2.618 effort=50 velocity=14
- added joint left_toe_joint: type fixed, parent left_foot_link, child left_toe_link, origin xyz=0.152 0 0 rpy=0 0 0, axis 0 1 0
- added joint left_wrist_yaw_joint: type fixed, parent left_elbow_link, child left_wrist_yaw_link, origin xyz=0.138 0 -0.017415 rpy=0 0 0, axis 1 0 0, limit lower=-2.618 upper=2.618 effort=50 velocity=14
- added joint right_ankle_pitch_joint: type revolute, parent right_knee_link, child right_ankle_pitch_link, origin xyz=0 0 -0.34 rpy=0 0 0, axis 0 1 0, limit lower=-0.873 upper=0.524 effort=50 velocity=15
- added joint right_ankle_roll_joint: type revolute, parent right_ankle_pitch_link, child right_ankle_roll_link, origin xyz=0 0 -0.018 rpy=0 0 0, axis 1 0 0, limit lower=-0.262 upper=0.262 effort=50 velocity=15
- added joint right_elbow_joint: type fixed, parent right_shoulder_yaw_link, child right_elbow_link, origin xyz=0.01924 0 -0.0979 rpy=0 1 0, axis 0 1 0, limit lower=-0.96 upper=2.0944 effort=50 velocity=14
- added joint right_foot_joint: type fixed, parent right_ankle_roll_link, child right_foot_link, origin xyz=0.000000 0.000000 -0.044760000 rpy=0 0 0, axis 0 0 1
- added joint right_hand_palm_joint: type fixed, parent right_wrist_yaw_link, child right_hand_palm_link, origin xyz=0.138 0.000000 0.0 rpy=0 0 0, axis 0 0 1
- added joint right_hip_pitch_joint: type revolute, parent pelvis, child right_hip_pitch_link, origin xyz=0 -0.06875 0 rpy=0 0 0, axis 0 1 0, limit lower=-2.7925 upper=2.7925 effort=120 velocity=20
- added joint right_hip_roll_joint: type revolute, parent right_hip_pitch_link, child right_hip_roll_link, origin xyz=0 -0.053724 -0.045579 rpy=0 0 0, axis 1 0 0, limit lower=-2.967 upper=0.524 effort=120 velocity=20
- added joint right_hip_yaw_joint: type revolute, parent right_hip_roll_link, child right_hip_yaw_link, origin xyz=-0.00050599 0.0029213 -0.12555 rpy=0 0 0, axis 0 0 1, limit lower=-2.7925 upper=2.7925 effort=120 velocity=20
- added joint right_knee_joint: type revolute, parent right_hip_yaw_link, child right_knee_link, origin xyz=-0.052111 0 -0.13729 rpy=0 0 0, axis 0 1 0, limit lower=0 upper=2.653 effort=120 velocity=20
- added joint right_shoulder_pitch_joint: type fixed, parent torso_link, child right_shoulder_pitch_link, origin xyz=0 -0.11963 0.3208 rpy=0 0.2 0, axis 0 0.99255 -0.12187, limit lower=-2.88 upper=2.88 effort=50 velocity=14
- added joint right_shoulder_roll_joint: type fixed, parent right_shoulder_pitch_link, child right_shoulder_roll_link, origin xyz=0 -0.047187 -0.013786 rpy=-0.15 0 0, axis 1 0 0, limit lower=-2.2515 upper=0.175 effort=50 velocity=14
- added joint right_shoulder_yaw_joint: type fixed, parent right_shoulder_roll_link, child right_shoulder_yaw_link, origin xyz=0 0 -0.1171 rpy=0 0 0, axis 0 0 1, limit lower=-2.618 upper=2.618 effort=50 velocity=14
- added joint right_toe_joint: type fixed, parent right_foot_link, child right_toe_link, origin xyz=0.152 0 0 rpy=0 0 0, axis 1 0 0
- added joint right_wrist_yaw_joint: type fixed, parent right_elbow_link, child right_wrist_yaw_link, origin xyz=0.138 0 -0.017415 rpy=0 0 0, axis 1 0 0, limit lower=-2.618 upper=2.618 effort=50 velocity=14
- added joint waist_yaw_joint: type fixed, parent pelvis, child torso_link, origin xyz=0 0 0.0619 rpy=0 0 0, axis 0 0 1, limit lower=-2.79 upper=2.79 effort=120 velocity=20
